File: Diseño/EEG.brd (EAGLE design)
At the start: 100 x 80 mm, 32 parts, among them IC1 REF2033AIDDCT, IC2 MCP73831T-2ACI_OT, IC3 LP38692MP-3.3_NOPB, X1 MINI-USB_4P-85-32004-40X

Commit message: correcciones
Parts:
- removed X1: MINI-USB_4P-85-32004-40X, con-cypressindustries:85-32004-40X
- added J1: USB3500-30-A-KIT, USB3500-30-A-KIT:USB350030AKIT
- added J2: SJ3-35083A-TR, SJ3-35083A-TR:SJ335083ATR
Connections:
- new net CS1: INA_1.1, J2.2
- new net CS2: INA_1.4, J2.5
- net +BATT: no longer X1.1
- net GND: now also J1.MH1, J1.MH2, J1.MH3, J1.MH4, J2.1; no longer X1.4
Changed lines of the file:
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@@
 <attribute name="VALUE" x="16.51" y="31.75" size="1.27" layer="27" align="center"/>
 </element>
-<element name="X1" library="con-cypressindustries" library_urn="urn:adsk.eagle:library:138" package="85-32004-40X" package3d_urn="urn:adsk.eagle:package:6444/1" value="MINI-USB_4P-85-32004-40X" x="30.48" y="8.89" smashed="yes">
-<attribute name="MF" value="" x="88.9" y="1.27" size="1.778" layer="27" display="off"/>
-<attribute name="MPN" value="" x="88.9" y="1.27" size="1.778" layer="27" display="off"/>
-<attribute name="NAME" x="25.98" y="14.39" size="1.27" layer="25"/>
-<attribute name="OC_FARNELL" value="unknown" x="88.9" y="1.27" size="1.778" layer="27" display="off"/>
-<attribute name="OC_NEWARK" value="unknown" x="88.9" y="1.27" size="1.778" layer="27" display="off"/>
-<attribute name="POPULARITY" value="0" x="88.9" y="1.27" size="1.778" layer="27" display="off"/>
-<attribute name="VALUE" x="23.44" y="1.89" size="1.27" layer="27"/>
+<element name="J1" library="USB3500-30-A-KIT" package="USB350030AKIT" value="USB3500-30-A-KIT" x="6.985" y="-5.715" smashed="yes">
+<attribute name="DESCRIPTION" value="USB Connectors Micro B Skt, Mid Mount-SMT, R/A, 30u&quot;, With Peg, T&amp;R, IP67 + USBTJ-02 Gasket" x="6.985" y="-5.715" size="1.778" layer="27" display="off"/>
+<attribute name="HEIGHT" value="2.8mm" x="6.985" y="-5.715" size="1.778" layer="27" display="off"/>
+<attribute name="MANUFACTURER_NAME" value="GCT (GLOBAL CONNECTOR TECHNOLOGY)" x="6.985" y="-5.715" size="1.778" layer="27" display="off"/>
+<attribute name="MANUFACTURER_PART_NUMBER" value="USB3500-30-A-KIT" x="6.985" y="-5.715" size="1.778" layer="27" display="off"/>
+<attribute name="MOUSER_PART_NUMBER" value="640-USB3500-30-A-KIT" x="6.985" y="-5.715" size="1.778" layer="27" display="off"/>
+<attribute name="MOUSER_PRICE-STOCK" value="https://www.mouser.co.uk/ProductDetail/GCT/USB3500-30-A-KIT?qs=KUoIvG%2F9IlZmD2kH2DfgYg%3D%3D" x="6.985" y="-5.715" size="1.778" layer="27" display="off"/>
+<attribute name="NAME" x="6.985" y="-4.565" size="1.27" layer="25" align="center"/>
+<attribute name="VALUE" x="6.985" y="-4.565" size="1.27" layer="27" align="center"/>
+</element>
+<element name="J2" library="SJ3-35083A-TR" package="SJ335083ATR" value="SJ3-35083A-TR" x="5.08" y="-16.51" smashed="yes">
+<attribute name="DESCRIPTION" value="3.5 mm Stereo Jack, Through Hole, 3 Conductors, 0 Internal Switches,  Tape &amp; Reel Packaging" x="5.08" y="-16.51" size="1.778" layer="27" display="off"/>
+<attribute name="HEIGHT" value="5.3mm" x="5.08" y="-16.51" size="1.778" layer="27" display="off"/>
+<attribute name="MANUFACTURER_NAME" value="Same Sky" x="5.08" y="-16.51" size="1.778" layer="27" display="off"/>
+<attribute name="MANUFACTURER_PART_NUMBER" value="SJ3-35083A-TR" x="5.08" y="-16.51" size="1.778" layer="27" display="off"/>
+<attribute name="MOUSER_PART_NUMBER" value="179-SJ3-35083A-TR" x="5.08" y="-16.51" size="1.778" layer="27" display="off"/>
+<attribute name="MOUSER_PRICE-STOCK" value="https://www.mouser.co.uk/ProductDetail/Same-Sky/SJ3-35083A-TR?qs=IKkN%2F947nfAXbylC140wLg%3D%3D" x="5.08" y="-16.51" size="1.778" layer="27" display="off"/>
+<attribute name="NAME" x="8.68" y="-14.095" size="1.27" layer="25" align="center"/>
+<attribute name="VALUE" x="8.68" y="-14.095" size="1.27" layer="27" align="center"/>
 </element>
 </elements>
@@
 <contactref element="R2" pad="1"/>
 <contactref element="C3" pad="2"/>
-<contactref element="X1" pad="4"/>
 <contactref element="IC3" pad="5"/>
 <contactref element="INA_1" pad="5"/>
@@
 <contactref element="LOW_PASS_1" pad="2"/>
 <contactref element="ESP32-S3" pad="1"/>
+<contactref element="J1" pad="MH1"/>
+<contactref element="J1" pad="MH2"/>
+<contactref element="J1" pad="MH3"/>
+<contactref element="J1" pad="MH4"/>
+<contactref element="J2" pad="1"/>
 <wire x1="87.53" y1="63.71" x2="96.38" y2="70.03" width="0" layer="19" extent="1-1"/>
 <wire x1="87.53" y1="62.31" x2="87.53" y2="63.71" width="0" layer="19" extent="1-1"/>
@@
 <wire x1="8.28" y1="34.93" x2="14.48" y2="48.26" width="0" layer="19" extent="1-1"/>
 <wire x1="8.28" y1="26.03" x2="8.28" y2="34.93" width="0" layer="19" extent="1-1"/>
-<wire x1="31.73" y1="7.09" x2="29.865" y2="29.845" width="0" layer="19" extent="1-1"/>
+<wire x1="11.835" y1="-3.215" x2="8.28" y2="26.03" width="0" layer="19" extent="1-1"/>
+<wire x1="11.835" y1="-5.715" x2="11.835" y2="-3.215" width="0" layer="19" extent="1-1"/>
+<wire x1="2.135" y1="-5.715" x2="11.835" y2="-5.715" width="0" layer="19" extent="1-1"/>
+<wire x1="2.135" y1="-3.215" x2="2.135" y2="-5.715" width="0" layer="19" extent="1-1"/>
+<wire x1="5.08" y1="-16.51" x2="2.135" y2="-5.715" width="0" layer="19" extent="1-1"/>
 </signal>
 <signal name="N$1">
@@
 </signal>
 <signal name="+BATT">
-<contactref element="X1" pad="1"/>
 <contactref element="C3" pad="1"/>
 <contactref element="IC2" pad="3"/>
-<wire x1="32.02" y1="69.85" x2="31.73" y2="10.69" width="0" layer="19" extent="1-1"/>
 <wire x1="29.865" y1="28.895" x2="32.02" y2="69.85" width="0" layer="19" extent="1-1"/>
 </signal>
@@
 <wire x1="78.88" y1="66.22" x2="20" y2="74.93" width="0" layer="19" extent="1-1"/>
 </signal>
+<signal name="CS1">
+<contactref element="INA_1" pad="1"/>
+<contactref element="J2" pad="2"/>
+<wire x1="14.38" y1="-16.51" x2="4.908" y2="69.215" width="0" layer="19" extent="1-1"/>
+</signal>
+<signal name="CS2">
+<contactref element="INA_1" pad="4"/>
+<contactref element="J2" pad="5"/>
+<wire x1="6.98" y1="-11.41" x2="4.908" y2="65.405" width="0" layer="19" extent="1-1"/>
+</signal>
 </signals>

Commit message: Se actualizo el diagrama de la ESP 32-S3
Parts:
- added C4: 0.1 uF, rcl:C0805
Connections:
- net GND: now also C4.1, S2.3, S3.4; no longer S2.1, S3.3
- net N$13: now also C4.2, S3.2; no longer S3.1
- net N$15: now also S2.1; no longer S2.3
Changed lines of the file:
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@@
 <attribute name="VALUE" x="8.68" y="-14.095" size="1.27" layer="27" align="center"/>
+</element>
+<element name="C4" library="rcl" library_urn="urn:adsk.eagle:library:334" package="C0805" package3d_urn="urn:adsk.eagle:package:23617/2" value="0.1 uF" x="1.27" y="-22.86" smashed="yes">
+<attribute name="NAME" x="0" y="-21.59" size="1.27" layer="25"/>
+<attribute name="POPULARITY" value="88" x="1.27" y="-22.86" size="1.778" layer="27" display="off"/>
+<attribute name="SPICEPREFIX" value="C" x="1.27" y="-22.86" size="1.778" layer="27" display="off"/>
+<attribute name="VALUE" x="0" y="-25.4" size="1.27" layer="27"/>
 </element>
 </elements>
@@
 <contactref element="C1_HP2" pad="2"/>
 <contactref element="C1_HP3" pad="1"/>
-<contactref element="S2" pad="1"/>
-<contactref element="S3" pad="3"/>
 <contactref element="ESP32-S3" pad="40"/>
 <contactref element="ESP32-S3" pad="41"/>
@@
 <contactref element="J1" pad="MH4"/>
 <contactref element="J2" pad="1"/>
+<contactref element="S2" pad="3"/>
+<contactref element="C4" pad="1"/>
+<contactref element="S3" pad="4"/>
 <wire x1="87.53" y1="63.71" x2="96.38" y2="70.03" width="0" layer="19" extent="1-1"/>
 <wire x1="87.53" y1="62.31" x2="87.53" y2="63.71" width="0" layer="19" extent="1-1"/>
@@
 <wire x1="29.865" y1="29.845" x2="26.055" y2="36.83" width="0" layer="19" extent="1-1"/>
 <wire x1="14.48" y1="48.26" x2="24.785" y2="48.895" width="0" layer="19" extent="1-1"/>
+<wire x1="14.58" y1="34.93" x2="26.055" y2="36.83" width="0" layer="19" extent="1-1"/>
+<wire x1="8.28" y1="22.23" x2="14.58" y2="34.93" width="0" layer="19" extent="1-1"/>
 <wire x1="7.005" y1="60.325" x2="14.48" y2="48.26" width="0" layer="19" extent="1-1"/>
 <wire x1="10.332" y1="65.405" x2="7.005" y2="60.325" width="0" layer="19" extent="1-1"/>
-<wire x1="8.28" y1="34.93" x2="14.48" y2="48.26" width="0" layer="19" extent="1-1"/>
-<wire x1="8.28" y1="26.03" x2="8.28" y2="34.93" width="0" layer="19" extent="1-1"/>
-<wire x1="11.835" y1="-3.215" x2="8.28" y2="26.03" width="0" layer="19" extent="1-1"/>
+<wire x1="11.835" y1="-3.215" x2="8.28" y2="22.23" width="0" layer="19" extent="1-1"/>
 <wire x1="11.835" y1="-5.715" x2="11.835" y2="-3.215" width="0" layer="19" extent="1-1"/>
 <wire x1="2.135" y1="-5.715" x2="11.835" y2="-5.715" width="0" layer="19" extent="1-1"/>
 <wire x1="2.135" y1="-3.215" x2="2.135" y2="-5.715" width="0" layer="19" extent="1-1"/>
 <wire x1="5.08" y1="-16.51" x2="2.135" y2="-5.715" width="0" layer="19" extent="1-1"/>
+<wire x1="0.32" y1="-22.86" x2="5.08" y2="-16.51" width="0" layer="19" extent="1-1"/>
 </signal>
 <signal name="N$1">
@@
 <contactref element="ESP32-S3" pad="3"/>
 <contactref element="R1_HP2" pad="1"/>
-<contactref element="S2" pad="3"/>
-<wire x1="8.28" y1="22.23" x2="78.88" y2="67.49" width="0" layer="19" extent="1-1"/>
-<wire x1="49.215" y1="53.34" x2="8.28" y2="22.23" width="0" layer="19" extent="1-1"/>
+<contactref element="S2" pad="1"/>
+<wire x1="49.215" y1="53.34" x2="78.88" y2="67.49" width="0" layer="19" extent="1-1"/>
 <wire x1="51.115" y1="46.99" x2="49.215" y2="53.34" width="0" layer="19" extent="1-1"/>
-</signal>
-<signal name="N$13">
-<contactref element="S3" pad="1"/>
-<contactref element="R1_HP3" pad="1"/>
-<contactref element="ESP32-S3" pad="27"/>
-<wire x1="39.055" y1="46.99" x2="8.28" y2="38.73" width="0" layer="19" extent="1-1"/>
-<wire x1="96.38" y1="53.52" x2="8.28" y2="38.73" width="0" layer="19" extent="1-1"/>
+<wire x1="8.28" y1="26.03" x2="51.115" y2="46.99" width="0" layer="19" extent="1-1"/>
 </signal>
 <signal name="O4">
@@
 <wire x1="6.98" y1="-11.41" x2="4.908" y2="65.405" width="0" layer="19" extent="1-1"/>
 </signal>
+<signal name="N$13">
+<contactref element="ESP32-S3" pad="27"/>
+<contactref element="C4" pad="2"/>
+<contactref element="R1_HP3" pad="1"/>
+<contactref element="S3" pad="2"/>
+<wire x1="39.055" y1="46.99" x2="96.38" y2="53.52" width="0" layer="19" extent="1-1"/>
+<wire x1="14.58" y1="38.73" x2="39.055" y2="46.99" width="0" layer="19" extent="1-1"/>
+<wire x1="2.22" y1="-22.86" x2="14.58" y2="38.73" width="0" layer="19" extent="1-1"/>
+</signal>
 </signals>

Commit message: mod circuito de carga, amplificadores y filtros
Parts:
- C1_HP1, C1_LP1, C2_HP1: value 10uF -> 100nF
- C2: value 5uF -> 100nF
- R1_HP1: value 1.6k -> 230k
- R1_LP1, R2_LP1: value 450 -> 33k
- R2_HP1: value 3.2k -> 230k
- RF_AMP1: value 10k -> 51k
Connections:
- removed net N$1: C1.1, IC2.4, LED1.A
- net +5V: now also C1.1, C3.1, IC2.4, J1.1, LED1.A
- net +BATT: now also S1.B1; no longer C3.1
- net GND: now also J1.5
Changed lines of the file:
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@@
 <attribute name="VALUE" x="32.655" y="65.41" size="1.016" layer="27"/>
 </element>
-<element name="C1_HP1" library="rcl" library_urn="urn:adsk.eagle:library:334" package="C0805" package3d_urn="urn:adsk.eagle:package:23617/2" value="10uF" x="48.895" y="73.025" smashed="yes">
+<element name="C1_HP1" library="rcl" library_urn="urn:adsk.eagle:library:334" package="C0805" package3d_urn="urn:adsk.eagle:package:23617/2" value="100nF" x="48.895" y="73.025" smashed="yes">
 <attribute name="NAME" x="47.625" y="74.295" size="1.27" layer="25"/>
 <attribute name="POPULARITY" value="88" x="76.835" y="17.145" size="1.778" layer="27" display="off"/>
@@
 <attribute name="VALUE" x="48.895" y="44.45" size="1.27" layer="27"/>
 </element>
-<element name="C1_LP1" library="rcl" library_urn="urn:adsk.eagle:library:334" package="C0805" package3d_urn="urn:adsk.eagle:package:23617/2" value="10uF" x="7.62" y="74.93" smashed="yes">
+<element name="C1_LP1" library="rcl" library_urn="urn:adsk.eagle:library:334" package="C0805" package3d_urn="urn:adsk.eagle:package:23617/2" value="100nF" x="7.62" y="74.93" smashed="yes">
 <attribute name="NAME" x="6.35" y="76.2" size="1.27" layer="25"/>
 <attribute name="POPULARITY" value="88" x="71.12" y="19.05" size="1.778" layer="27" display="off"/>
@@
 <attribute name="VALUE" x="6.35" y="72.39" size="1.27" layer="27"/>
 </element>
-<element name="C2" library="rcl" library_urn="urn:adsk.eagle:library:334" package="C0805" package3d_urn="urn:adsk.eagle:package:23617/2" value="5uF" x="34.925" y="60.96" smashed="yes">
+<element name="C2" library="rcl" library_urn="urn:adsk.eagle:library:334" package="C0805" package3d_urn="urn:adsk.eagle:package:23617/2" value="100nF" x="34.925" y="60.96" smashed="yes">
 <attribute name="NAME" x="33.655" y="62.23" size="1.27" layer="25"/>
 <attribute name="POPULARITY" value="88" x="56.515" y="-1.27" size="1.778" layer="27" display="off"/>
@@
 <attribute name="VALUE" x="33.655" y="58.42" size="1.27" layer="27"/>
 </element>
-<element name="C2_HP1" library="rcl" library_urn="urn:adsk.eagle:library:334" package="C0805" package3d_urn="urn:adsk.eagle:package:23617/2" value="10uF" x="19.05" y="62.865" smashed="yes">
+<element name="C2_HP1" library="rcl" library_urn="urn:adsk.eagle:library:334" package="C0805" package3d_urn="urn:adsk.eagle:package:23617/2" value="100nF" x="19.05" y="62.865" smashed="yes">
 <attribute name="NAME" x="17.78" y="64.135" size="1.27" layer="25"/>
 <attribute name="POPULARITY" value="88" x="73.66" y="6.985" size="1.778" layer="27" display="off"/>
@@
 <attribute name="VALUE" x="40.64" y="51.435" size="1.27" layer="27"/>
 </element>
-<element name="R1_HP1" library="rcl" library_urn="urn:adsk.eagle:library:334" package="R0805" package3d_urn="urn:adsk.eagle:package:23553/2" value="1.6k" x="48.26" y="66.675" smashed="yes">
+<element name="R1_HP1" library="rcl" library_urn="urn:adsk.eagle:library:334" package="R0805" package3d_urn="urn:adsk.eagle:package:23553/2" value="230k" x="48.26" y="66.675" smashed="yes">
 <attribute name="NAME" x="47.625" y="67.945" size="1.27" layer="25"/>
 <attribute name="POPULARITY" value="86" x="78.74" y="17.145" size="1.778" layer="27" display="off"/>
@@
 <attribute name="VALUE" x="39.37" y="44.45" size="1.27" layer="27"/>
 </element>
-<element name="R1_LP1" library="rcl" library_urn="urn:adsk.eagle:library:334" package="R0805" package3d_urn="urn:adsk.eagle:package:23553/2" value="450" x="19.685" y="69.215" smashed="yes">
+<element name="R1_LP1" library="rcl" library_urn="urn:adsk.eagle:library:334" package="R0805" package3d_urn="urn:adsk.eagle:package:23553/2" value="33k" x="19.685" y="69.215" smashed="yes">
 <attribute name="NAME" x="16.51" y="70.485" size="1.27" layer="25"/>
 <attribute name="POPULARITY" value="86" x="85.725" y="19.685" size="1.778" layer="27" display="off"/>
@@
 <attribute name="VALUE" x="40.64" y="64.135" size="1.27" layer="27"/>
 </element>
-<element name="R2_HP1" library="rcl" library_urn="urn:adsk.eagle:library:334" package="R0805" package3d_urn="urn:adsk.eagle:package:23553/2" value="3.2k" x="19.05" y="57.15" smashed="yes">
+<element name="R2_HP1" library="rcl" library_urn="urn:adsk.eagle:library:334" package="R0805" package3d_urn="urn:adsk.eagle:package:23553/2" value="230k" x="19.05" y="57.15" smashed="yes">
 <attribute name="NAME" x="18.415" y="58.42" size="1.27" layer="25"/>
 <attribute name="POPULARITY" value="86" x="76.2" y="7.62" size="1.778" layer="27" display="off"/>
@@
 <attribute name="VALUE" x="18.415" y="54.61" size="1.27" layer="27"/>
 </element>
-<element name="R2_LP1" library="rcl" library_urn="urn:adsk.eagle:library:334" package="R0805" package3d_urn="urn:adsk.eagle:package:23553/2" value="450" x="34.29" y="55.245" smashed="yes">
+<element name="R2_LP1" library="rcl" library_urn="urn:adsk.eagle:library:334" package="R0805" package3d_urn="urn:adsk.eagle:package:23553/2" value="33k" x="34.29" y="55.245" smashed="yes">
 <attribute name="NAME" x="33.655" y="56.515" size="1.27" layer="25"/>
 <attribute name="POPULARITY" value="86" x="53.34" y="-0.635" size="1.778" layer="27" display="off"/>
@@
 <attribute name="VALUE" x="33.655" y="52.705" size="1.27" layer="27"/>
 </element>
-<element name="RF_AMP1" library="rcl" library_urn="urn:adsk.eagle:library:334" package="R0805" package3d_urn="urn:adsk.eagle:package:23553/2" value="10k" x="19.05" y="74.93" smashed="yes">
+<element name="RF_AMP1" library="rcl" library_urn="urn:adsk.eagle:library:334" package="R0805" package3d_urn="urn:adsk.eagle:package:23553/2" value="51k" x="19.05" y="74.93" smashed="yes">
 <attribute name="NAME" x="18.415" y="76.2" size="1.27" layer="25"/>
 <attribute name="POPULARITY" value="86" x="86.36" y="33.02" size="1.778" layer="27" display="off"/>
@@
 <contactref element="J1" pad="MH4"/>
 <contactref element="J2" pad="1"/>
-<contactref element="S2" pad="3"/>
 <contactref element="C4" pad="1"/>
 <contactref element="S3" pad="4"/>
+<contactref element="J1" pad="5"/>
+<contactref element="S2" pad="3"/>
 <wire x1="87.53" y1="63.71" x2="96.38" y2="70.03" width="0" layer="19" extent="1-1"/>
 <wire x1="87.53" y1="62.31" x2="87.53" y2="63.71" width="0" layer="19" extent="1-1"/>
@@
 <wire x1="7.005" y1="60.325" x2="14.48" y2="48.26" width="0" layer="19" extent="1-1"/>
 <wire x1="10.332" y1="65.405" x2="7.005" y2="60.325" width="0" layer="19" extent="1-1"/>
-<wire x1="11.835" y1="-3.215" x2="8.28" y2="22.23" width="0" layer="19" extent="1-1"/>
+<wire x1="8.285" y1="-1.915" x2="8.28" y2="22.23" width="0" layer="19" extent="1-1"/>
+<wire x1="11.835" y1="-3.215" x2="8.285" y2="-1.915" width="0" layer="19" extent="1-1"/>
 <wire x1="11.835" y1="-5.715" x2="11.835" y2="-3.215" width="0" layer="19" extent="1-1"/>
-<wire x1="2.135" y1="-5.715" x2="11.835" y2="-5.715" width="0" layer="19" extent="1-1"/>
-<wire x1="2.135" y1="-3.215" x2="2.135" y2="-5.715" width="0" layer="19" extent="1-1"/>
+<wire x1="2.135" y1="-3.215" x2="8.285" y2="-1.915" width="0" layer="19" extent="1-1"/>
+<wire x1="2.135" y1="-5.715" x2="2.135" y2="-3.215" width="0" layer="19" extent="1-1"/>
 <wire x1="5.08" y1="-16.51" x2="2.135" y2="-5.715" width="0" layer="19" extent="1-1"/>
 <wire x1="0.32" y1="-22.86" x2="5.08" y2="-16.51" width="0" layer="19" extent="1-1"/>
-</signal>
-<signal name="N$1">
-<contactref element="LED1" pad="A"/>
-<contactref element="IC2" pad="4"/>
-<contactref element="C1" pad="1"/>
-<wire x1="32.655" y1="67.31" x2="32.365" y2="28.895" width="0" layer="19" extent="1-1"/>
-<wire x1="34.925" y1="73.245" x2="32.655" y2="67.31" width="0" layer="19" extent="1-1"/>
 </signal>
 <signal name="N$3">
@@
 </signal>
 <signal name="+BATT">
-<contactref element="C3" pad="1"/>
 <contactref element="IC2" pad="3"/>
-<wire x1="29.865" y1="28.895" x2="32.02" y2="69.85" width="0" layer="19" extent="1-1"/>
+<contactref element="S1" pad="B1"/>
+<wire x1="11.97" y1="15.05" x2="29.865" y2="28.895" width="0" layer="19" extent="1-1"/>
 </signal>
 <signal name="N$11">
@@
 <signal name="+5V">
 <contactref element="S1" pad="D1"/>
+<contactref element="LED1" pad="A"/>
+<contactref element="IC2" pad="4"/>
+<contactref element="C1" pad="1"/>
+<contactref element="J1" pad="1"/>
+<contactref element="C3" pad="1"/>
+<wire x1="32.02" y1="69.85" x2="34.925" y2="73.245" width="0" layer="19" extent="1-1"/>
+<wire x1="32.655" y1="67.31" x2="32.02" y2="69.85" width="0" layer="19" extent="1-1"/>
+<wire x1="32.365" y1="28.895" x2="32.655" y2="67.31" width="0" layer="19" extent="1-1"/>
+<wire x1="17.97" y1="15.05" x2="32.365" y2="28.895" width="0" layer="19" extent="1-1"/>
+<wire x1="5.685" y1="-1.915" x2="17.97" y2="15.05" width="0" layer="19" extent="1-1"/>
 </signal>
 <signal name="N$9">
